Commit message: sharpa: fix right-hand body frame asymmetry via post-joint rotation

File: dexmachina/assets/sharpa_hand/right_sharpa_wave_6dof.urdf (robot description, URDF)
Before this commit: robot right_sharpa_wave, 40 links, 39 joints
Links:
- added link R_wrist_pre_link, mass 0.001
Joints:
- added joint R_wrist_rotation_joint: type fixed, parent R_wrist_pre_link, child right_hand_C_MC, origin xyz=0 0 0 rpy=0 0 3.14159265
- joint R_forearm_yaw_link_joint: child right_hand_C_MC -> R_wrist_pre_link
